File: ESP32C3_RF_Test.kicad_sch (KiCad schematic)
At the start: 55 parts, among them J1 Conn_I2C, J2 Conn_UART, J3 USB_C_Receptacle, J4 Conn_Ext_3v3, SW1 SW_RST, SW2 SW_BOOT, U1 ESP32-C3, U2 RT9013-33GB, Y1 Crystal_40MHz

Commit message: BOM change
Parts:
- U1: value ESP32-C3 -> ESP32-C3FH4
Changed lines of the file:
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@@
     (in_bom yes) (on_board yes) (fields_autoplaced)
     (property "Reference" "U1" (id 0) (at 128.27 35.56 0))
-    (property "Value" "ESP32-C3" (id 1) (at 128.27 38.1 0))
+    (property "Value" "ESP32-C3FH4" (id 1) (at 128.27 38.1 0))
     (property "Footprint" "Package_DFN_QFN:QFN-32-1EP_5x5mm_P0.5mm_EP3.1x3.1mm_ThermalVias" (id 2) (at 128.27 101.6 0)
       (effects (font (size 1.27 1.27)) hide)
@@
     )
     (path "/f15de1c3-f77c-45c8-87bd-22e63a7159ab"
-      (reference "U1") (unit 1) (value "ESP32-C3") (footprint "Package_DFN_QFN:QFN-32-1EP_5x5mm_P0.5mm_EP3.1x3.1mm_ThermalVias")
+      (reference "U1") (unit 1) (value "ESP32-C3FH4") (footprint "Package_DFN_QFN:QFN-32-1EP_5x5mm_P0.5mm_EP3.1x3.1mm_ThermalVias")
     )
     (path "/2ad833bb-132a-4e56-9c22-3b599638690c"
